Commit message: Updated husky_ur5 config files to reflect parts added
Specifically the ur5_arm_camera_mount_link and ur5_arm_laser_pointer_link

File: husky_description/urdf/husky_ur5.urdf (robot description, URDF)
Before this commit: robot husky, 30 links, 29 joints
Links:
- removed link ur5_arm_marker_link
- removed link ur5_arm_tool_mount_link
- added link camera_optical_frame
- added link ur5_arm_camera_mount_link; collision mesh filename=package://ur_description/meshes/ur5/collision/camera_mount.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 scale=0.001 0.001 0.001; visual mesh filename=package://ur_description/meshes/ur5/visual/camera_mount.dae scale=0.001 0.001 0.001
- added link ur5_arm_camera_optical_frame
- added link ur5_arm_laser_pointer_link; collision mesh filename=package://ur_description/meshes/ur5/collision/laser_pointer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 scale=0.001 0.001 0.001; visual mesh filename=package://ur_description/meshes/ur5/visual/laser_pointer.dae scale=0.001 0.001 0.001
- link ur5_arm_camera_link: geometry collision mesh filename=package://ur_description/meshes/ur5/collision/camera.stl scale=0.001 0.001 0.001; visual mesh filename=package://ur_description/meshes/ur5/visual/camera.dae scale=0.001 0.001 0.001
Joints:
- removed joint kinect_frame_joint
- removed joint ur5_arm_marker_joint
- removed joint ur5_arm_tool_mount_joint
- added joint camera_optical_joint: type fixed, parent camera_link, child camera_optical_frame, origin xyz=0 0 0 rpy=-1.57079632679 0 -1.57079632679
- added joint kinectv2_frame_joint: type fixed, parent camera_mount_link, child camera_link, origin xyz=0.0 0.095 0.11 rpy=0.0 0.0 3.14159265359
- added joint ur5_arm_camera_mount_joint: type fixed, parent ur5_arm_wrist_3_link, child ur5_arm_camera_mount_link, origin xyz=0.0 0.0823 0.0 rpy=0.0 0.0 1.570796325
- added joint ur5_arm_camera_optical_joint: type fixed, parent ur5_arm_camera_link, child ur5_arm_camera_optical_frame, origin xyz=0.0 0.0 0.0 rpy=-1.5708 0.0 -1.5708
- added joint ur5_arm_laser_pointer_joint: type fixed, parent ur5_arm_camera_mount_link, child ur5_arm_laser_pointer_link, origin xyz=0.157 0.0 0.0 rpy=0.0 0.0 0.0
- joint imu_joint: origin xyz=0.19 0 0.149 rpy=0 -1.5708 3.1416 -> xyz=0.19 0 0.149 rpy=0 -1.5708 3.14159265359
- joint sensor_arch_mount: origin xyz=-0.35 0.0 0.51 rpy=0.0 0.0 -3.14 -> xyz=-0.35 0.0 0.51 rpy=0.0 0.0 -3.14159265359
- joint ur5_arm_camera_joint: origin xyz=0.11 0.0 0.055 rpy=0.0 0.0 0.0 -> xyz=.056433755002348 0.0 0.069206449979048 rpy=0.0 0.29984756549263 0.0; parent ur5_arm_tool_mount_link -> ur5_arm_camera_mount_link
