Commit message: Added an intermediate link between camera_link and kinect2_link

File: husky_description/urdf/husky.urdf.xacro (robot description, xacro)
@@ -188,10 +188,16 @@
         </collision>
       </link>
-      <joint name="kinectv2_frame_joint" type="fixed">
+      <joint name="camera_link_joint" type="fixed">
         <origin xyz="0.028 -0.096 0.112" rpy="0.0 0.0 0.0" />
         <parent link="camera_mount_link"/>
+        <child link="camera_link"/>
+      </joint>
+      <link name="kinect2_link" />
+      <joint name="kinect2_link_joint" type="fixed">
+        <origin xyz="0.0 0.0 0.0" rpy="-1.57079632679 0 -1.57079632679" />
+        <parent link="camera_link"/>
         <child link="kinect2_link"/>
       </joint>
-      <xacro:kinectv2_camera prefix="kinect2"/>
+      <xacro:kinectv2_camera prefix="camera"/>
     </xacro:if>
     <!-- Spawn Primesense Carmine 1.09 if primesense_enabled = "true" -->
