Commit message: Added primesence camera and added optical_joint to urdf from gazebo cons

File: husky_description/urdf/accessories/kinect_camera.urdf.xacro (robot description, xacro)
@@ -38,4 +38,5 @@
       </visual>
       <collision>
+	<origin xyz="0 0 0" rpy="0 0 ${M_PI/2}"/>
         <geometry>
           <box size="0.07 0.3 0.09"/>

File: husky_description/urdf/accessories/kinectv2_camera.urdf.xacro (robot description, xacro)
@@ -25,8 +25,8 @@
 SOFTWARE, EVEN IF ADVISED OF THE POSSIBILITY OF SUCH DAMAGE.
 -->
-<robot xmlns:xacro="http://ros.org/wiki/xacro" name="kinect_camera">
+<robot xmlns:xacro="http://ros.org/wiki/xacro" name="kinectv2_camera">
   <xacro:macro name="kinectv2_camera" params="prefix:=camera">
     <!-- Create kinect reference frame -->
-    <!-- Add mesh for kinect -->
+    <!-- Add mesh for kinectv2 -->
     <link name="${prefix}_link">
       <visual>

File: husky_description/urdf/husky.urdf.xacro (robot description, xacro)
@@ -27,4 +27,5 @@
   <xacro:include filename="$(find husky_description)/urdf/accessories/kinect_camera.urdf.xacro"/>
   <xacro:include filename="$(find husky_description)/urdf/accessories/kinectv2_camera.urdf.xacro"/>
+  <xacro:include filename="$(find husky_description)/urdf/accessories/primesense_carmine_1-09_camera.urdf.xacro"/>
   <xacro:include filename="$(find husky_description)/urdf/accessories/sick_lms1xx_mount.urdf.xacro"/>
   <xacro:include filename="$(find husky_description)/urdf/accessories/sensor_arch.urdf.xacro"/>
@@ -88,5 +89,5 @@
     <link name="imu_link"/>
     <joint name="imu_joint" type="fixed">
-      <origin xyz="$(optenv HUSKY_IMU_XYZ 0.19 0 0.149)" rpy="$(optenv HUSKY_IMU_RPY 0 -1.5708 3.1416)" />
+      <origin xyz="$(optenv HUSKY_IMU_XYZ 0.19 0 0.149)" rpy="$(optenv HUSKY_IMU_RPY 0 -1.57079632679 3.14159265359)" />
       <parent link="base_link" />
       <child link="imu_link" />
@@ -116,5 +117,5 @@
         <parent link="top_plate_link" />
         <child link="ur5_arm_base_link" />
-        <origin xyz="0.3058 0 0.0065" rpy="0.0 0.0 -1.57" />
+        <origin xyz="0.3058 0 0.0065" rpy="0.0 0.0 -1.57079632679" />
       </joint>
     </xacro:if>
@@ -127,7 +128,8 @@
         <parent link="top_plate_link" />
         <child link="ur5_arm_base_link" />
-        <origin xyz="0.3058 0 0.0065" rpy="0.0 0.0 -1.57" />
-      </joint>
-    </xacro:if>
+        <origin xyz="0.3058 0 0.0065" rpy="0.0 0.0 -1.57079632679" />
+      </joint>
+    </xacro:if>
+    <!-- Spawn LIDAR if laser_enabled = "true" -->
     <xacro:if value="$(arg laser_enabled)">
       <sick_lms1xx_mount prefix="base" topic="scan"/>
@@ -139,18 +141,26 @@
       </joint>
     </xacro:if>
+    <!-- Spawn Kinect if kinect_enabled = "true" -->
     <xacro:if value="$(arg kinect_enabled)">
       <xacro:sensor_arch prefix="" parent="top_plate_link">
-        <origin xyz="-0.35 0 0.51" rpy="0 0 -3.14"/>
+        <origin xyz="-0.35 0 0.51" rpy="0 0 -3.14159265359"/>
       </xacro:sensor_arch>
       <joint name="kinect_frame_joint" type="fixed">
-        <origin xyz="$(optenv HUSKY_KINECT_XYZ 0 0 0)" rpy="$(optenv HUSKY_KINECT_RPY 0 0.18 3.14)" />
+        <origin xyz="$(optenv HUSKY_KINECT_XYZ 0 0 0)" rpy="$(optenv HUSKY_KINECT_RPY 0 0.18 3.14159265359)" />
         <parent link="sensor_arch_mount_link"/>
         <child link="camera_link"/>
       </joint>
       <xacro:kinect_camera prefix="camera"/>
-    </xacro:if>
+      <link name="camera_optical_frame"/>
+      <joint name="camera_optical_joint" type="fixed">
+        <origin xyz="0 0 0" rpy="-1.57079632679 0 -1.57079632679"/>
+        <parent link="camera_link"/>
+        <child link="camera_optical_frame"/>
+      </joint>
+    </xacro:if>
+    <!-- Spawn KinectV2 if kinectv2_enabled = "true" -->
     <xacro:if value="$(arg kinectv2_enabled)">
       <xacro:sensor_arch prefix="" parent="top_plate_link">
-        <origin xyz="-0.35 0.0 0.51" rpy="0.0 0.0 -3.14"/>
+        <origin xyz="-0.35 0.0 0.51" rpy="0.0 0.0 -3.14159265359"/>
       </xacro:sensor_arch>
       <!-- Attach the camera mount to the sensor arch -->
@@ -163,5 +173,5 @@
       <link name="camera_mount_link">
         <visual>
-          <origin xyz="0.0 0.0 0.0" rpy="1.57 0.0 1.57"/>
+          <origin xyz="0.0 0.0 0.0" rpy="1.57079632679 0.0 1.57079632679"/>
           <geometry>
             <mesh filename="package://husky_description/meshes/accessories/kinectv2_mount.dae" />
@@ -172,5 +182,5 @@
         </visual>
         <collision>
-          <origin xyz="0.0 0.0 0.0" rpy="1.57 0.0 1.57"/>
+          <origin xyz="0.0 0.0 0.0" rpy="1.57079632679 0.0 1.57079632679"/>
           <geometry>
             <mesh filename="package://husky_description/meshes/accessories/kinectv2_mount.stl" />
@@ -178,10 +188,52 @@
         </collision>
       </link>
-      <joint name="kinect_frame_joint" type="fixed">
-        <origin xyz="$(optenv HUSKY_KINECT_XYZ 0.0 0.095 0.11)" rpy="$(optenv HUSKY_KINECT_RPY 0.0 0.18 3.14)" />
+      <joint name="kinectv2_frame_joint" type="fixed">
+        <origin xyz="0.0 0.095 0.11" rpy="0.0 0.0 3.14159265359" />
         <parent link="camera_mount_link"/>
         <child link="camera_link"/>
       </joint>
       <xacro:kinectv2_camera prefix="camera"/>
+      <link name="camera_optical_frame"/>
+      <joint name="camera_optical_joint" type="fixed">
+        <origin xyz="0 0 0" rpy="-1.57079632679 0 -1.57079632679"/>
+        <parent link="camera_link"/>
+        <child link="camera_optical_frame"/>
+      </joint>
+    </xacro:if>
+    <!-- Spawn Primesense Carmine 1.09 if primesense_enabled = "true" -->
+    <xacro:if value="$(arg primesense_enabled)">
+      <xacro:sensor_arch prefix="" parent="top_plate_link">
+        <origin xyz="-0.35 0 0.51" rpy="0 0 -3.14159265359"/>
+      </xacro:sensor_arch>
+      <joint name="primesense_camera_joint" type="fixed">
+        <origin xyz="-0.020 0 0.0343994" rpy="0.0 0.0 3.14159265359" />
+        <parent link="sensor_arch_mount_link"/>
+        <child link="camera_link"/>
+      </joint>
+      <xacro:primesense_camera prefix="camera"/>
+      <link name="camera_rgb_frame" />
+      <joint name="camera_rgb_joint" type="fixed">
+        <origin rpy="0 0 0" xyz="0 0.02 0" />
+        <parent link="camera_link" />
+        <child link="camera_rgb_frame" />
+      </joint>
+      <link name="camera_rgb_optical_frame" />
+      <joint name="camera_rgb_optical_joint" type="fixed">
+        <origin rpy="-1.57079632679 0 -1.57079632679" xyz="0 0 0" />
+        <parent link="camera_rgb_frame" />
+        <child link="camera_rgb_optical_frame" />
+      </joint>
+      <link name="camera_depth_frame" />
+      <joint name="camera_depth_joint" type="fixed">
+        <origin rpy="0 0 0" xyz="0 0.045 0" />
+        <parent link="camera_link" />
+        <child link="camera_depth_frame" />
+      </joint>
+      <link name="camera_depth_optical_frame" />
+      <joint name="camera_depth_optical_joint" type="fixed">
+        <origin rpy="-1.57079632679 0 -1.57079632679" xyz="0 0 0" />
+        <parent link="camera_depth_frame" />
+        <child link="camera_depth_optical_frame" />
+      </joint>
     </xacro:if>
   </xacro:macro>
