Commit message: Update KinectV2 position and link name

File: husky_description/urdf/accessories/kinectv2_camera.urdf.xacro (robot description, xacro)
@@ -26,10 +26,10 @@
 -->
 <robot xmlns:xacro="http://ros.org/wiki/xacro" name="kinectv2_camera">
-  <xacro:macro name="kinectv2_camera" params="prefix:=camera">
+  <xacro:macro name="kinectv2_camera" params="prefix:=kinect2">
     <!-- Create kinect reference frame -->
     <!-- Add mesh for kinectv2 -->
     <link name="${prefix}_link">
       <visual>
-        <origin xyz="0.0 0.095 -0.04" rpy="0 0 ${-1*M_PI/2}"/>
+        <origin xyz="-0.028 0.096 -0.042" rpy="0 0 -1.57079632679"/>
         <geometry>
           <mesh filename="package://husky_description/meshes/accessories/kinectv2.dae" />
@@ -37,5 +37,5 @@
       </visual>
       <collision>
-        <origin xyz="0.0 0.095 -0.04" rpy="0 0 ${-1*M_PI/2}"/>
+        <origin xyz="-0.028 0.096 -0.042" rpy="0 0 -1.57079632679"/>
         <geometry>
           <mesh filename="package://husky_description/meshes/accessories/kinectv2.stl" />

File: husky_description/urdf/husky.urdf.xacro (robot description, xacro)
@@ -166,5 +166,5 @@
       <!-- Attach the camera mount to the sensor arch -->
       <joint name="camera_mount_joint" type="fixed">
-           <origin xyz="0.0 0.0 0.0" rpy="0.0 0.0 0.0"/>
+           <origin xyz="0.0 0.0 0.0" rpy="0.0 0.0 3.14159265359"/>
            <parent link="sensor_arch_mount_link"/>
            <child link="camera_mount_link"/>
@@ -189,15 +189,9 @@
       </link>
       <joint name="kinectv2_frame_joint" type="fixed">
-        <origin xyz="0.0 0.095 0.11" rpy="0.0 0.0 3.14159265359" />
+        <origin xyz="0.028 -0.096 0.112" rpy="0.0 0.0 0.0" />
         <parent link="camera_mount_link"/>
-        <child link="camera_link"/>
-      </joint>
-      <xacro:kinectv2_camera prefix="camera"/>
-      <link name="camera_optical_frame"/>
-      <joint name="camera_optical_joint" type="fixed">
-        <origin xyz="0 0 0" rpy="-1.57079632679 0 -1.57079632679"/>
-        <parent link="camera_link"/>
-        <child link="camera_optical_frame"/>
-      </joint>
+        <child link="kinect2_link"/>
+      </joint>
+      <xacro:kinectv2_camera prefix="kinect2"/>
     </xacro:if>
     <!-- Spawn Primesense Carmine 1.09 if primesense_enabled = "true" -->
