Commit message: Added ccam specific hardware, updated configs and collision DAEs to STLs

File: husky_description/urdf/accessories/sick_lms1xx_mount.urdf.xacro (robot description, xacro)
@@ -31,5 +31,5 @@
     <link name="${prefix}_laser_mount">
       <visual>
-        <origin xyz="0 0 0" rpy="0 0 ${-M_PI/2}" />
+        <origin xyz="0 0 0" rpy="${M_PI} 0 ${-M_PI/2}" />
         <geometry>
           <!-- Origin of this mesh is the base of the bracket. -->
@@ -38,5 +38,5 @@
       </visual>
       <collision>
-        <origin xyz="0 0 .0585" rpy="0 0 0" />
+        <origin xyz="0 0 .0585" rpy="${M_PI} 0 ${-M_PI/2}" />
         <geometry>
           <box size=".1 .108 .117" />
@@ -46,5 +46,5 @@
     <joint name="${prefix}_laser_joint" type="fixed">
       <!-- This offset is from the base of the bracket to the LIDAR's focal point. -->
-      <origin xyz="0.0352 0 0.0566" rpy="${M_PI} 0 0" />
+      <origin xyz="-0.0352 0 -0.0566" rpy="${M_PI} 0 0" />
       <parent link="${prefix}_laser_mount" />
       <child link="${prefix}_laser" />

File: husky_description/urdf/description.xacro (robot description, xacro)
@@ -24,5 +24,7 @@
   <xacro:arg name="laser_enabled" default="false" />
   <xacro:arg name="ur5_enabled" default="false" />
+  <xacro:arg name="ur5_camera_enabled" default="false" />
   <xacro:arg name="kinect_enabled" default="false" />
+  <xacro:arg name="kinectv2_enabled" default="false" />
   <xacro:include filename="$(find husky_description)/urdf/husky.urdf.xacro" />
   <xacro:husky_robot />

File: husky_description/urdf/husky.urdf.xacro (robot description, xacro)
@@ -26,4 +26,5 @@
   <xacro:include filename="$(find husky_description)/urdf/wheel.urdf.xacro" />
   <xacro:include filename="$(find husky_description)/urdf/accessories/kinect_camera.urdf.xacro"/>
+  <xacro:include filename="$(find husky_description)/urdf/accessories/kinectv2_camera.urdf.xacro"/>
   <xacro:include filename="$(find husky_description)/urdf/accessories/sick_lms1xx_mount.urdf.xacro"/>
   <xacro:include filename="$(find husky_description)/urdf/accessories/sensor_arch.urdf.xacro"/>
@@ -73,7 +74,7 @@
     <link name="inertial_link">
       <inertial>
-        <mass value="33.455" />
+        <mass value="60" />
         <origin xyz="-0.08748 -0.00085 0.09947" />
-        <inertia ixx="0.6022" ixy="-0.02364" ixz="-0.1197" iyy="1.7386" iyz="-0.001544" izz="2.0296" />
+        <inertia ixx="1.08995475113" ixy="-0.0427873303" ixz="-0.2166515837" iyy="3.14678733031" iyz="-0.00279457012" izz="3.67348416289" />
       </inertial>
     </link>
@@ -118,8 +119,19 @@
       </joint>
     </xacro:if>
+    <xacro:if value="$(arg ur5_camera_enabled)">
+      <xacro:property name="reflect" value="-1" />
+      <!-- Spawn arm -->
+      <xacro:ur5_robot prefix="ur5_arm_" joint_limited="true"/>
+      <!-- Join arm -->
+      <joint name="ur5_arm_base" type="fixed">
+        <parent link="top_plate_link" />
+        <child link="ur5_arm_base_link" />
+        <origin xyz="0.3058 0 0.0065" rpy="0.0 0.0 -1.57" />
+      </joint>
+    </xacro:if>
     <xacro:if value="$(arg laser_enabled)">
       <sick_lms1xx_mount prefix="base" topic="scan"/>
       <joint name="laser_mount_joint" type="fixed">
-        <origin xyz="$(optenv HUSKY_LMS1XX_XYZ 0.2206 0.0 0.00635)"
+        <origin xyz="$(optenv HUSKY_LMS1XX_XYZ 0.415 0.0 -0.04)"
                 rpy="$(optenv HUSKY_LMS1XX_RPY 0.0 0.0 0.0)" />
         <parent link="top_plate_link" />
@@ -138,4 +150,39 @@
       <xacro:kinect_camera prefix="camera"/>
     </xacro:if>
+    <xacro:if value="$(arg kinectv2_enabled)">
+      <xacro:sensor_arch prefix="" parent="top_plate_link">
+        <origin xyz="-0.35 0.0 0.51" rpy="0.0 0.0 -3.14"/>
+      </xacro:sensor_arch>
+      <!-- Attach the camera mount to the sensor arch -->
+      <joint name="camera_mount_joint" type="fixed">
+           <origin xyz="0.0 0.0 0.0" rpy="0.0 0.0 0.0"/>
+           <parent link="sensor_arch_mount_link"/>
+           <child link="camera_mount_link"/>
+      </joint>
+      <!-- Spawn the kinectv2 mount link -->
+      <link name="camera_mount_link">
+        <visual>
+          <origin xyz="0.0 0.0 0.0" rpy="1.57 0.0 1.57"/>
+          <geometry>
+            <mesh filename="package://husky_description/meshes/accessories/kinectv2_mount.dae" />
+          </geometry>
+          <material name="LightGrey">
+            <color rgba="0.2 0.2 0.2 1.0"/>
+          </material>
+        </visual>
+        <collision>
+          <origin xyz="0.0 0.0 0.0" rpy="1.57 0.0 1.57"/>
+          <geometry>
+            <mesh filename="package://husky_description/meshes/accessories/kinectv2_mount.stl" />
+          </geometry>
+        </collision>
+      </link>
+      <joint name="kinect_frame_joint" type="fixed">
+        <origin xyz="$(optenv HUSKY_KINECT_XYZ 0.0 0.095 0.11)" rpy="$(optenv HUSKY_KINECT_RPY 0.0 0.18 3.14)" />
+        <parent link="camera_mount_link"/>
+        <child link="camera_link"/>
+      </joint>
+      <xacro:kinectv2_camera prefix="camera"/>
+    </xacro:if>
   </xacro:macro>
 </robot>

File: husky_description/urdf/wheel.urdf.xacro (robot description, xacro)
@@ -43,6 +43,6 @@
 		</link>
 		<gazebo reference="${wheel_prefix}_wheel_link">
-			<mu1 value="1.0"/>
-			<mu2 value="1.0"/>
+			<mu1 value="0.025"/>
+			<mu2 value="0.025"/>
 			<kp value="10000000.0" />
 			<kd value="1.0" />

Commit message: Fixed lidar orientation

File: husky_description/urdf/accessories/sick_lms1xx_mount.urdf.xacro (robot description, xacro)
@@ -31,5 +31,5 @@
     <link name="${prefix}_laser_mount">
       <visual>
-        <origin xyz="0 0 0" rpy="${M_PI} 0 ${-M_PI/2}" />
+        <origin xyz="0 0 0" rpy="0 ${-M_PI} ${-M_PI/2}" />
         <geometry>
           <!-- Origin of this mesh is the base of the bracket. -->
@@ -38,5 +38,5 @@
       </visual>
       <collision>
-        <origin xyz="0 0 .0585" rpy="${M_PI} 0 ${-M_PI/2}" />
+        <origin xyz="0 0 .0585" rpy="0 ${-M_PI} ${-M_PI/2}" />
         <geometry>
           <box size=".1 .108 .117" />
@@ -46,5 +46,5 @@
     <joint name="${prefix}_laser_joint" type="fixed">
       <!-- This offset is from the base of the bracket to the LIDAR's focal point. -->
-      <origin xyz="-0.0352 0 -0.0566" rpy="${M_PI} 0 0" />
+      <origin xyz="-0.0352 0 -0.0566" rpy="0 0 0" />
       <parent link="${prefix}_laser_mount" />
       <child link="${prefix}_laser" />
